Commit message: feat(slam): 优化SLAM配置并添加雷达数据过滤
- 调整SLAM参数以适应低速机器人，降低最小更新距离/角度
- 添加雷达数据过滤配置，滤除车身遮挡区域
- 更新启动脚本以包含ekf_odom包
- 修改URDF使雷达和相机关节可旋转
- 更新保存地图脚本以使用相对路径
- 在uart节点中添加雷达和相机关节状态

File: src/butter_robot_description/urdf/butter_robot.urdf (robot description, URDF)
Before this commit: robot 黄油机器人总装.SLDASM, 8 links, 7 joints
Joints:
- joint camera_joint: axis 0 0 0 -> 0 0 1; limit (none) -> lower=0 upper=0 effort=0 velocity=0; type fixed -> revolute
- joint radar_joint: axis 0 0 0 -> 0 0 1; limit (none) -> lower=0 upper=0 effort=0 velocity=0; type fixed -> revolute

Commit message: feat: 启用音频和视觉相关节点并优化配置
- 启用audio_asr、audio_rkllm和audio_tts节点
- 启用视觉管道容器(rk_camera+rk_inference+rk_streamer)
- 修改audio_rkllm.launch.py中force_english参数为False
- 简化uart/main.py中的JointState发布逻辑
- 更新butter_robot.urdf中雷达和相机关节类型为fixed
- 修改audio_tts.launch.py中的语音参数(音色ID和方言)
- 新增.trae/rules目录下的多份规则文档
- 新增.trae/skills目录下的技能文档
- 更新all_launch.launch.py集成所有功能节点

File: src/butter_robot_description/urdf/butter_robot.urdf (robot description, URDF)
Before this commit: robot 黄油机器人总装.SLDASM, 8 links, 7 joints
Joints:
- joint camera_joint: axis 0 0 1 -> 0 0 0; limit lower=0 upper=0 effort=0 velocity=0 -> (none); type revolute -> fixed
- joint radar_joint: axis 0 0 1 -> 0 0 0; limit lower=0 upper=0 effort=0 velocity=0 -> (none); type revolute -> fixed
